File: hardware/ bottom_board/ bottom_board.kicad_pcb (KiCad board)
At the start: 2 copper layers, 86 x 62 mm, 3 parts

Commit message: more work on code
Other:
- board text added: "To save position, long press a button for 3s: A: servo1 only B, C: both servos D: servo2 only To recall saved position, press and release button To return to normal operation, press and release same button again"
- board text added: "v1.0-beta2, May 2024"
Changed lines of the file:
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@@
     (effects (font (size 1.5 1.5) (thickness 0.2)) (justify bottom))
+  )
+  (gr_text "v1.0-beta2, May 2024" (at 163.5 117.75) (layer "F.SilkS")
+    (effects (font (size 1.5 1.5) (thickness 0.2)) (justify bottom))
+  )
+  (gr_text "To save position, long press a button for 3s:\nA: servo1 only\nB, C: both servos\nD: servo2 only \nTo recall saved position, press and release button\nTo return to normal operation, press and release same button again " (at 122 91.25) (layer "F.SilkS")
+    (effects (font (size 1 1) (thickness 0.15)) (justify left bottom))
   )
   (gr_text "Servo controller" (at 140.25 74.25) (layer "F.SilkS")

Commit message: kicad files update
Other:
- board text added: "To save position, long press a button for 3s: A: servo1 only B, C: both servos D: servo2 only To recall saved position, press and release button To return to normal operation, press and release same button again Uses 4 AA batteries. To replace batteries, remove this panel"
- board text added: "v1.0-beta2, June 2024"
- board text removed: "To save position, long press a button for 3s: A: servo1 only B, C: both servos D: servo2 only To recall saved position, press and release button To return to normal operation, press and release same button again"
- board text removed: "v1.0-beta2, May 2024"
Changed lines of the file:
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@@
     (effects (font (size 1.5 1.5) (thickness 0.2)) (justify bottom))
   )
-  (gr_text "v1.0-beta2, May 2024" (at 163.5 117.75) (layer "F.SilkS")
+  (gr_text "v1.0-beta2, June 2024" (at 163.5 117.75) (layer "F.SilkS")
     (effects (font (size 1.5 1.5) (thickness 0.2)) (justify bottom))
   )
-  (gr_text "To save position, long press a button for 3s:\nA: servo1 only\nB, C: both servos\nD: servo2 only \nTo recall saved position, press and release button\nTo return to normal operation, press and release same button again " (at 122 91.25) (layer "F.SilkS")
-    (effects (font (size 1 1) (thickness 0.15)) (justify left bottom))
+  (gr_text "To save position, long press a button for 3s:\n  A: servo1 only\n  B, C: both servos\n  D: servo2 only \nTo recall saved position, press and release button\nTo return to normal operation, press and release \nsame button again \n\nUses 4 AA batteries. \nTo replace batteries,  remove this panel" (at 117.4 104.4) (layer "F.SilkS")
+    (effects (font (size 1.4 1.4) (thickness 0.2) bold) (justify left bottom))
   )
   (gr_text "Servo controller" (at 140.25 74.25) (layer "F.SilkS")

Commit message: adding QR code
Parts:
- added G***: LOGO, shurik-personal:servo_controller_qr, F.Cu at (167.9, 75.2)
- moved G*** 7.11 mm to (135.2, 69.8)
Other:
- board text added: "To save position, long press a button for 2s: A: servo1 only B, C: both servos D: servo2 only To recall saved position, press and release button To return to normal operation, press and release same button again Uses 4 AA batteries. To replace batteries, remove this panel"
- board text added: "servo-controller.rtfd.io"
- board text removed: "To save position, long press a button for 3s: A: servo1 only B, C: both servos D: servo2 only To recall saved position, press and release button To return to normal operation, press and release same button again Uses 4 AA batteries. To replace batteries, remove this panel"
- board text removed: "servo_controller.rtfd.io"

Commit message: board update
Parts:
- removed the G*** at (135.2, 69.8)
- removed the G*** at (167.9, 75.2)
- added G***: LOGO, shurik-personal:4137-logo-small, F.Cu at (167.9, 75.2)
- added G***: LOGO, shurik-personal:servo-controller-tindie, F.Cu at (112.2, 75.2)
Other:
- board text added: "designed by FTC 4137 Islandbots"
- board text added: "tindie.com/stores/irobotics"
- board text added: "v1.0.0, June 2024"
- board text removed: "by Island Robotics"
- board text removed: "servo-controller.rtfd.io"
- board text removed: "v1.0-beta2, June 2024"
