File: hardware/mainboard/mainboard.kicad_sch (KiCad schematic)
At the start: 21 parts, among them J1 Conn_01x02, J2 Conn_01x03, J3 Conn_01x03, SW1 SW_SPST, SW2 SW_SPST, SW3 SW_SPST, SW4 SW_SPDT, SW5 SW_SPST, U1 TXB0104PWR, U2 SN74LVC2G241DCY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

Commit message: getting ready for beta2
Parts:
- removed J1: Conn_01x02, Connector_PinHeader_2.54mm:PinHeader_1x02_P2.54mm_Vertical, symbol Connector_Generic:Conn_01x02
- removed U5: LM1117MP-5.0, Package_TO_SOT_SMD:SOT-223-3_TabPin2, symbol Regulator_Linear:LM1117MP-5.0
- added C5: 220uF, Capacitor_SMD:CP_Elec_6.3x7.7, symbol Device:C_Polarized_US
- added D1: D_Schottky, Diode_SMD:D_SOD-323, symbol Device:D_Schottky
- added J1, J2: Conn_01x01, shurik-personal:connector-1p-generic-nosilk, symbol Connector_Generic:Conn_01x01
- C3: value 10uF -> 22uF; footprint Capacitor_SMD:C_0603_1608Metric -> Capacitor_SMD:C_0805_2012Metric; LCSC C14663 -> C45783
- C5: LCSC (none) -> C131158
- SW2: renamed from SW1; LCSC C2885087 -> C2885143
- SW3: renamed from SW2; LCSC C2885087 -> C2885143
- SW4: renamed from SW3; LCSC C2885087 -> C2885143
- SW5: LCSC C2885087 -> C2885143
- renumbered J2 to J3, J3 to J4, R2 to R1, R3 to R2, R1 to R3, SW4 to SW1
Connections:
- net +5V: now also D1.1 (K)
- net GND: now also C5.2, J2.1 (Pin_1)
- net RXD: now also U2.6 (1Y); no longer U2.2 (1A)
- net SERVO1L: now also U2.2 (1A); no longer U2.6 (1Y), U3.6 (11)
- net VCC: now also C5.1, D1.2 (A)
- net at SW1.2 (B): now also J1.1 (Pin_1)
- net CTRRL renamed CTRL
Other:
- moved on the sheet: C3, C5, J3, J4, R1, R2, R3, RV1, RV2, SW1, U1

Commit message: more work on code
Parts:
- added J5: Conn_01x05, Connector_PinSocket_2.54mm:PinSocket_1x05_P2.54mm_Vertical, symbol Connector_Generic:Conn_01x05
Connections:
- net +5V: now also J5.2 (Pin_2)
- net GND: now also J5.5 (Pin_5)
- net SERVO1: now also J5.3 (Pin_3)
- net SERVO1L: now also J5.4 (Pin_4)
- net VCC: now also J5.1 (Pin_1)
Changed lines of the file:
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@@
+    (stroke (width 0) (type default))
+  )
+  (wire (pts (xy 55.88 170.18) (xy 55.88 173.99))
     (stroke (width 0) (type default))
   )
@@
     (stroke (width 0) (type default))
   )
+  (wire (pts (xy 58.42 162.56) (xy 49.53 162.56))
+    (stroke (width 0) (type default))
+  )
   (polyline (pts (xy 161.29 67.31) (xy 142.24 67.31))
     (stroke (width 0) (type default))
@@
     (stroke (width 0) (type default))
   )
+  (wire (pts (xy 49.53 165.1) (xy 58.42 165.1))
+    (stroke (width 0) (type default))
+  )
   (wire (pts (xy 36.83 36.83) (xy 54.61 36.83))
     (stroke (width 0) (type default))
   )
+  (wire (pts (xy 58.42 160.02) (xy 55.88 160.02))
+    (stroke (width 0) (type default))
+  )
   (wire (pts (xy 240.03 31.75) (xy 240.03 27.94))
     (stroke (width 0) (type default))
@@
     (stroke (width 0) (type default))
   )
+  (wire (pts (xy 49.53 162.56) (xy 49.53 157.48))
+    (stroke (width 0) (type default))
+  )
   (wire (pts (xy 119.38 96.52) (xy 119.38 100.33))
     (stroke (width 0) (type default))
@@
     (stroke (width 0) (type default))
   )
+  (wire (pts (xy 58.42 170.18) (xy 55.88 170.18))
+    (stroke (width 0) (type default))
+  )
   (wire (pts (xy 60.96 116.84) (xy 73.66 116.84))
     (stroke (width 0) (type default))
@@
     (stroke (width 0) (type default))
   )
+  (wire (pts (xy 55.88 160.02) (xy 55.88 157.48))
+    (stroke (width 0) (type default))
+  )
   (wire (pts (xy 63.5 34.29) (xy 63.5 36.83))
     (stroke (width 0) (type default))
@@
   )
   (wire (pts (xy 143.51 20.32) (xy 149.86 20.32))
+    (stroke (width 0) (type default))
+  )
+  (wire (pts (xy 49.53 167.64) (xy 58.42 167.64))
     (stroke (width 0) (type default))
   )
@@
     (effects (font (size 1.27 1.27)) (justify right bottom))
   )
+  (label "SERVO1" (at 49.53 165.1 0) (fields_autoplaced)
+    (effects (font (size 1.27 1.27)) (justify left bottom))
+  )
   (label "SERVO2L" (at 102.87 41.91 0) (fields_autoplaced)
     (effects (font (size 1.27 1.27)) (justify left bottom))
@@
   )
   (label "SERVO1" (at 170.18 35.56 0) (fields_autoplaced)
+    (effects (font (size 1.27 1.27)) (justify left bottom))
+  )
+  (label "SERVO1L" (at 49.53 167.64 0) (fields_autoplaced)
     (effects (font (size 1.27 1.27)) (justify left bottom))
   )
@@
         (path "/ec64e276-e8ff-4b7e-81d1-2720aa338102"
           (reference "#PWR019") (unit 1)
+        )
+      )
+    )
+  )
+  (symbol (lib_id "power:GND") (at 55.88 173.99 0) (unit 1)
+    (in_bom yes) (on_board yes) (dnp no) (fields_autoplaced)
+    (property "Reference" "#PWR024" (at 55.88 180.34 0)
+      (effects (font (size 1.27 1.27)) hide)
+    )
+    (property "Value" "GND" (at 55.88 179.07 0)
+      (effects (font (size 1.27 1.27)))
+    )
+    (property "Footprint" "" (at 55.88 173.99 0)
+      (effects (font (size 1.27 1.27)) hide)
+    )
+    (property "Datasheet" "" (at 55.88 173.99 0)
+      (effects (font (size 1.27 1.27)) hide)
+    )
+    (pin "1")
+    (instances
+      (project "mainboard"
+        (path "/ec64e276-e8ff-4b7e-81d1-2720aa338102"
+          (reference "#PWR024") (unit 1)
         )
       )
@@
         (path "/ec64e276-e8ff-4b7e-81d1-2720aa338102"
           (reference "#PWR03") (unit 1)
+        )
+      )
+    )
+  )
+  (symbol (lib_id "power:+5V") (at 49.53 157.48 0) (unit 1)
+    (in_bom yes) (on_board yes) (dnp no) (fields_autoplaced)
+    (property "Reference" "#PWR026" (at 49.53 161.29 0)
+      (effects (font (size 1.27 1.27)) hide)
+    )
+    (property "Value" "+5V" (at 49.53 152.4 0)
+      (effects (font (size 1.27 1.27)))
+    )
+    (property "Footprint" "" (at 49.53 157.48 0)
+      (effects (font (size 1.27 1.27)) hide)
+    )
+    (property "Datasheet" "" (at 49.53 157.48 0)
+      (effects (font (size 1.27 1.27)) hide)
+    )
+    (pin "1")
+    (instances
+      (project "mainboard"
+        (path "/ec64e276-e8ff-4b7e-81d1-2720aa338102"
+          (reference "#PWR026") (unit 1)
         )
       )
@@
     )
   )
+  (symbol (lib_id "Connector_Generic:Conn_01x05") (at 63.5 165.1 0) (unit 1)
+    (in_bom yes) (on_board yes) (dnp no) (fields_autoplaced)
+    (property "Reference" "J5" (at 66.04 163.83 0)
+      (effects (font (size 1.27 1.27)) (justify left))
+    )
+    (property "Value" "Conn_01x05" (at 66.04 166.37 0)
+      (effects (font (size 1.27 1.27)) (justify left))
+    )
+    (property "Footprint" "Connector_PinSocket_2.54mm:PinSocket_1x05_P2.54mm_Vertical" (at 63.5 165.1 0)
+      (effects (font (size 1.27 1.27)) hide)
+    )
+    (property "Datasheet" "~" (at 63.5 165.1 0)
+      (effects (font (size 1.27 1.27)) hide)
+    )
+    (pin "1")
+    (pin "2")
+    (pin "3")
+    (pin "4")
+    (pin "5")
+    (instances
+      (project "mainboard"
+        (path "/ec64e276-e8ff-4b7e-81d1-2720aa338102"
+          (reference "J5") (unit 1)
+        )
+      )
+    )
+  )
   (symbol (lib_id "Switch:SW_SPST") (at 210.82 97.79 0) (unit 1)
     (in_bom yes) (on_board yes) (dnp no)
@@
         )
       )
+    )
+  )
+  (symbol (lib_id "power:VCC") (at 55.88 157.48 0) (unit 1)
+    (in_bom yes) (on_board yes) (dnp no) (fields_autoplaced)
+    (property "Reference" "#PWR025" (at 55.88 161.29 0)
+      (effects (font (size 1.27 1.27)) hide)
+    )
+    (property "Value" "VCC" (at 55.88 152.4 0)
+      (effects (font (size 1.27 1.27)))
+    )
+    (property "Footprint" "" (at 55.88 157.48 0)
+      (effects (font (size 1.27 1.27)) hide)
+    )
+    (property "Datasheet" "" (at 55.88 157.48 0)
+      (effects (font (size 1.27 1.27)) hide)
+    )
+    (pin "1")
+    (instances
+      (project "mainboard"
+        (path "/ec64e276-e8ff-4b7e-81d1-2720aa338102"
+          (reference "#PWR025") (unit 1)
+        )
+      )

Commit message: version 1.0.0
Parts:
- J3, J4, J5: LCSC (none) -> C49257
Changed lines of the file:
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@@
+      (effects (font (size 1.27 1.27)) hide)
+    )
+    (property "LCSC" "C49257" (at 203.2 36.83 0)
       (effects (font (size 1.27 1.27)) hide)
     )
@@
     )
     (property "Datasheet" "~" (at 182.88 38.1 0)
+      (effects (font (size 1.27 1.27)) hide)
+    )
+    (property "LCSC" "C49257" (at 185.42 36.83 0)
       (effects (font (size 1.27 1.27)) hide)
     )
@@
       (effects (font (size 1.27 1.27)) hide)
     )
+    (property "LCSC" "C49257" (at 66.04 163.83 0)
+      (effects (font (size 1.27 1.27)) hide)
+    )
